Commit message: Some cleanup and simulation setup

File: rover_description/urdf/rover.urdf (robot description, URDF)
Before this commit: robot rover, 16 links, 15 joints
Joints:
- joint AB-Rev: type continuous -> fixed
- joint AM-Rev: type continuous -> fixed
- joint AS1-Rev: type continuous -> fixed
- joint AS2-Rev: type continuous -> fixed
- joint AW-Rev: type continuous -> fixed
- joint BL-Rev: type continuous -> fixed
- joint BR-Rev: type continuous -> fixed
- joint RL-Rev: type continuous -> fixed
- joint RR-Rev: type continuous -> fixed
