Commit message: Working differential drive in gazebo with ros2 control

File: rover_description/urdf/rover.urdf.xacro (robot description, xacro)
@@ -4,4 +4,11 @@
   <!-- Import RRBot ros2_control description -->
   <xacro:include filename="rover.control.xacro" />
+  <link name="base_link"/>
+  <joint name="base_to_chassis" type="fixed">
+    <parent link="base_link"/>
+    <child link="Chassis"/>
+    <!-- Orient rover to face along +X axis -->
+    <origin xyz="0 0 0" rpy="0 0 -1.5708"/>
+  </joint>
   <link name="Chassis">
     <inertial>
@@ -92,5 +99,5 @@
       link="FL_Wheel" />
     <axis
-      xyz="0 0 1" />
+      xyz="0 0 -1" />
   </joint>
   <link name="FR_Wheel">
@@ -194,5 +201,5 @@
       link="BL_Wheel" />
     <axis
-      xyz="0 0 1" />
+      xyz="0 0 -1" />
   </joint>
   <link name="BR_Wheel">

Commit message: Use ZED for localization

File: rover_description/urdf/rover.urdf.xacro (robot description, xacro)
@@ -560,4 +560,13 @@
       xyz="0 1 0" />
   </joint>
+  <!-- <link name="Front_Zed_link"/>
+  <joint name="Front_Zed_link_joint" type="fixed">
+    <parent link="base_link"/>
+    <child link="Front_Zed_link"/>
+    <origin
+      xyz="0.55 0 -0.18"
+      rpy="0 0 0"
+    />
+  </joint> -->
   <xacro:rover_ros2_control use_gazebo="$(arg use_gazebo)"/>
   <xacro:if value="$(arg use_gazebo)">
@@ -577,8 +586,8 @@
     </xacro:zed_camera>
     <joint name="Front_Zed_joint" type="fixed">
-      <parent link="base_link"/>
-      <child link="Front_Zed_camera_link"/>
-      <origin
-        xyz="1 0 0"
+      <parent link="Front_Zed_camera_link"/>
+      <child link="base_link"/>
+      <origin
+        xyz="-0.55 0 0.18"
         rpy="0 0 0"
       />

Commit message: Zed imu/odom and gnss fusion for localization

File: rover_description/urdf/rover.urdf.xacro (robot description, xacro)
@@ -560,13 +560,4 @@
       xyz="0 1 0" />
   </joint>
-  <!-- <link name="Front_Zed_link"/>
-  <joint name="Front_Zed_link_joint" type="fixed">
-    <parent link="base_link"/>
-    <child link="Front_Zed_link"/>
-    <origin
-      xyz="0.55 0 -0.18"
-      rpy="0 0 0"
-    />
-  </joint> -->
   <xacro:rover_ros2_control use_gazebo="$(arg use_gazebo)"/>
   <xacro:if value="$(arg use_gazebo)">
@@ -586,8 +577,8 @@
     </xacro:zed_camera>
     <joint name="Front_Zed_joint" type="fixed">
-      <parent link="Front_Zed_camera_link"/>
-      <child link="base_link"/>
-      <origin
-        xyz="-0.55 0 0.18"
+      <parent link="base_link"/>
+      <child link="Front_Zed_camera_link"/>
+      <origin
+        xyz="0.55 0 -0.18"
         rpy="0 0 0"
       />
