Commit message: Fixed Gazebo Simulation Setup

File: rover_description/urdf/rover.control.xacro (robot description, xacro)
@@ -13,16 +13,38 @@
         <command_interface name="velocity"/>
         <state_interface name="velocity"/>
+        <state_interface name="position"/>
       </joint>
       <joint name="FR_Drive">
         <command_interface name="velocity"/>
         <state_interface name="velocity"/>
+        <state_interface name="position"/>
       </joint>
       <joint name="BL_Drive">
         <command_interface name="velocity"/>
         <state_interface name="velocity"/>
+        <state_interface name="position"/>
       </joint>
       <joint name="BR_Drive">
         <command_interface name="velocity"/>
         <state_interface name="velocity"/>
+        <state_interface name="position"/>
+      </joint>
+      <joint name="Arm_Base_Rotate">
+        <state_interface name="position"/>
+      </joint>
+      <joint name="Arm_Shoulder">
+        <state_interface name="position"/>
+      </joint>
+      <joint name="Arm_Elbow_Tilt">
+        <state_interface name="position"/>
+      </joint>
+      <joint name="Arm_Elbow_Rotate">
+        <state_interface name="position"/>
+      </joint>
+      <joint name="Arm_Wrist_Tilt">
+        <state_interface name="position"/>
+      </joint>
+      <joint name="Arm_Wrist_Rotate">
+        <state_interface name="position"/>
       </joint>
     </ros2_control>

File: rover_description/urdf/rover.urdf.xacro (robot description, xacro)
@@ -558,6 +558,8 @@
     <gazebo>
       <plugin filename="gz_ros2_control-system" name="gz_ros2_control::GazeboSimROS2ControlPlugin">
-        <parameters>../config/rover_controllers.yaml</parameters>
+        <parameters>$(find rover_description)/config/rover_controllers.yaml</parameters>
       </plugin>
+      <!-- Should probably optimize the collision shapes in the future -->
+      <self_collide>true</self_collide>
     </gazebo>
   </xacro:if>

Commit message: URDF updates and arm control plugin improvements

File: rover_description/urdf/rover.control.xacro (robot description, xacro)
@@ -57,5 +57,5 @@
         <!-- <command_interface name="velocity"/> -->
         <param name="epos_node_id">1</param>
-        <param name="position_target_scale">100.0</param>
+        <param name="position_target_scale">-2048.0</param>
       </joint>
       <joint name="Arm_Elbow_Tilt">
@@ -64,4 +64,6 @@
         <command_interface name="position"/>
         <!-- <command_interface name="velocity"/> -->
+        <param name="epos_node_id">2</param>
+        <param name="position_target_scale">-512.0</param>
       </joint>
       <joint name="Arm_Elbow_Rotate">
@@ -70,4 +72,6 @@
         <command_interface name="position"/>
         <!-- <command_interface name="velocity"/> -->
+        <param name="epos_node_id">3</param>
+        <param name="position_target_scale">44032.0</param>
       </joint>
       <joint name="Arm_Wrist_Tilt">
@@ -76,4 +80,7 @@
         <command_interface name="position"/>
         <!-- <command_interface name="velocity"/> -->
+        <param name="epos_node_id">4</param>
+        <param name="position_target_scale">512.0</param>
+        <param name="differential_index">0</param>
       </joint>
       <joint name="Arm_Wrist_Rotate">
@@ -82,4 +89,7 @@
         <command_interface name="position"/>
         <!-- <command_interface name="velocity"/> -->
+        <param name="epos_node_id">5</param>
+        <param name="position_target_scale">512.0</param>
+        <param name="differential_index">1</param>
       </joint>
     </ros2_control>

File: rover_description/urdf/rover.urdf.xacro (robot description, xacro)
@@ -571,3 +571,15 @@
     </gazebo>
   </xacro:if>
+  <xacro:unless value="$(arg use_gazebo)">
+    <xacro:include filename="$(find zed_wrapper)/urdf/zed_macro.urdf.xacro" />
+    <xacro:zed_camera name="Front_Zed" model="zed2i" baseline="0.0"/>
+    <joint name="Front_Zed_joint" type="fixed">
+      <parent link="base_link"/>
+      <child link="Front_Zed_camera_link"/>
+      <origin
+        xyz="1 0 0"
+        rpy="0 0 0"
+      />
+    </joint>
+  </xacro:unless>
 </robot>

Commit message: Add control+drivers for stepper motors

File: rover_description/urdf/rover.control.xacro (robot description, xacro)
@@ -36,5 +36,5 @@
       </joint>
     </ros2_control>
-    <ros2_control name="RoverArm" type="system">
+    <ros2_control name="RoverArmEPOS" type="system">
       <hardware>
         <xacro:if value="${use_gazebo}">
@@ -45,10 +45,10 @@
         </xacro:unless>
       </hardware>
-      <joint name="Arm_Base_Rotate">
+      <!-- <joint name="Arm_Base_Rotate">
         <state_interface name="position"/>
         <state_interface name="velocity"/>
         <command_interface name="position"/>
-        <!-- <command_interface name="velocity"/> -->
-      </joint>
+        <command_interface name="velocity"/>
+      </joint> -->
       <joint name="Arm_Shoulder">
         <state_interface name="position"/>
@@ -94,4 +94,22 @@
       </joint>
     </ros2_control>
+    <ros2_control name="RoverArmSteppers" type="system">
+      <hardware>
+        <xacro:if value="${use_gazebo}">
+          <plugin>gz_ros2_control/GazeboSimSystem</plugin>
+        </xacro:if>
+        <xacro:unless value="${use_gazebo}">
+          <plugin>rover_hardware/StepperSystem</plugin>
+        </xacro:unless>
+      </hardware>
+      <joint name="Arm_Base_Rotate">
+        <state_interface name="position"/>
+        <state_interface name="velocity"/>
+        <command_interface name="position"/>
+        <!-- <command_interface name="velocity"/> -->
+        <param name="topic_name">base_rotate</param>
+        <param name="tick_resolution">1000.0</param>
+      </joint>
+    </ros2_control>
   </xacro:macro>
 </robot>

Commit message: Update meshes and use coarse for collision

File: rover_description/urdf/rover.control.xacro (robot description, xacro)
@@ -109,5 +109,5 @@
         <!-- <command_interface name="velocity"/> -->
         <param name="topic_name">base_rotate</param>
-        <param name="tick_resolution">1000.0</param>
+        <param name="tick_resolution">-160000.0</param>
       </joint>
     </ros2_control>

File: rover_description/urdf/rover.urdf.xacro (robot description, xacro)
@@ -32,19 +32,19 @@
       <geometry>
         <mesh
-          filename="package://rover_description/meshes/Chassis.STL" />
-      </geometry>
-      <material
-        name="">
-        <color
-          rgba="0.752941176470588 0.752941176470588 0.752941176470588 1" />
-      </material>
-    </visual>
-    <collision>
-      <origin
-        xyz="0 0 0"
-        rpy="0 0 0" />
-      <geometry>
-        <mesh
-          filename="package://rover_description/meshes/Chassis.STL" />
+          filename="package://rover_description/meshes/fine/Chassis.STL" />
+      </geometry>
+      <material
+        name="">
+        <color
+          rgba="0.752941176470588 0.752941176470588 0.752941176470588 1" />
+      </material>
+    </visual>
+    <collision>
+      <origin
+        xyz="0 0 0"
+        rpy="0 0 0" />
+      <geometry>
+        <mesh
+          filename="package://rover_description/meshes/coarse/Chassis.STL" />
       </geometry>
     </collision>
@@ -71,19 +71,19 @@
       <geometry>
         <mesh
-          filename="package://rover_description/meshes/FL_Wheel.STL" />
-      </geometry>
-      <material
-        name="">
-        <color
-          rgba="0.752941176470588 0.752941176470588 0.752941176470588 1" />
-      </material>
-    </visual>
-    <collision>
-      <origin
-        xyz="0 0 0"
-        rpy="0 0 0" />
-      <geometry>
-        <mesh
-          filename="package://rover_description/meshes/FL_Wheel.STL" />
+          filename="package://rover_description/meshes/coarse/FL_Wheel.STL" />
+      </geometry>
+      <material
+        name="">
+        <color
+          rgba="0.752941176470588 0.752941176470588 0.752941176470588 1" />
+      </material>
+    </visual>
+    <collision>
+      <origin
+        xyz="0 0 0"
+        rpy="0 0 0" />
+      <geometry>
+        <mesh
+          filename="package://rover_description/meshes/coarse/FL_Wheel.STL" />
       </geometry>
     </collision>
@@ -122,19 +122,19 @@
       <geometry>
         <mesh
-          filename="package://rover_description/meshes/FR_Wheel.STL" />
-      </geometry>
-      <material
-        name="">
-        <color
-          rgba="0.752941176470588 0.752941176470588 0.752941176470588 1" />
-      </material>
-    </visual>
-    <collision>
-      <origin
-        xyz="0 0 0"
-        rpy="0 0 0" />
-      <geometry>
-        <mesh
-          filename="package://rover_description/meshes/FR_Wheel.STL" />
+          filename="package://rover_description/meshes/coarse/FR_Wheel.STL" />
+      </geometry>
+      <material
+        name="">
+        <color
+          rgba="0.752941176470588 0.752941176470588 0.752941176470588 1" />
+      </material>
+    </visual>
+    <collision>
+      <origin
+        xyz="0 0 0"
+        rpy="0 0 0" />
+      <geometry>
+        <mesh
+          filename="package://rover_description/meshes/coarse/FR_Wheel.STL" />
       </geometry>
     </collision>
@@ -173,19 +173,19 @@
       <geometry>
         <mesh
-          filename="package://rover_description/meshes/BL_Wheel.STL" />
-      </geometry>
-      <material
-        name="">
-        <color
-          rgba="0.752941176470588 0.752941176470588 0.752941176470588 1" />
-      </material>
-    </visual>
-    <collision>
-      <origin
-        xyz="0 0 0"
-        rpy="0 0 0" />
-      <geometry>
-        <mesh
-          filename="package://rover_description/meshes/BL_Wheel.STL" />
+          filename="package://rover_description/meshes/coarse/BL_Wheel.STL" />
+      </geometry>
+      <material
+        name="">
+        <color
+          rgba="0.752941176470588 0.752941176470588 0.752941176470588 1" />
+      </material>
+    </visual>
+    <collision>
+      <origin
+        xyz="0 0 0"
+        rpy="0 0 0" />
+      <geometry>
+        <mesh
+          filename="package://rover_description/meshes/coarse/BL_Wheel.STL" />
       </geometry>
     </collision>
@@ -224,19 +224,19 @@
       <geometry>
         <mesh
-          filename="package://rover_description/meshes/BR_Wheel.STL" />
-      </geometry>
-      <material
-        name="">
-        <color
-          rgba="0.752941176470588 0.752941176470588 0.752941176470588 1" />
-      </material>
-    </visual>
-    <collision>
-      <origin
-        xyz="0 0 0"
-        rpy="0 0 0" />
-      <geometry>
-        <mesh
-          filename="package://rover_description/meshes/BR_Wheel.STL" />
+          filename="package://rover_description/meshes/coarse/BR_Wheel.STL" />
+      </geometry>
+      <material
+        name="">
+        <color
+          rgba="0.752941176470588 0.752941176470588 0.752941176470588 1" />
+      </material>
+    </visual>
+    <collision>
+      <origin
+        xyz="0 0 0"
+        rpy="0 0 0" />
+      <geometry>
+        <mesh
+          filename="package://rover_description/meshes/coarse/BR_Wheel.STL" />
       </geometry>
     </collision>
@@ -275,19 +275,19 @@
       <geometry>
         <mesh
-          filename="package://rover_description/meshes/Arm_Base.STL" />
-      </geometry>
-      <material
-        name="">
-        <color
-          rgba="0.752941176470588 0.752941176470588 0.752941176470588 1" />
-      </material>
-    </visual>
-    <collision>
-      <origin
-        xyz="0 0 0"
-        rpy="0 0 0" />
-      <geometry>
-        <mesh
-          filename="package://rover_description/meshes/Arm_Base.STL" />
+          filename="package://rover_description/meshes/coarse/Arm_Base.STL" />
+      </geometry>
+      <material
+        name="">
+        <color
+          rgba="0.752941176470588 0.752941176470588 0.752941176470588 1" />
+      </material>
+    </visual>
+    <collision>
+      <origin
+        xyz="0 0 0"
+        rpy="0 0 0" />
+      <geometry>
+        <mesh
+          filename="package://rover_description/meshes/coarse/Arm_Base.STL" />
       </geometry>
     </collision>
@@ -326,19 +326,19 @@
       <geometry>
         <mesh
-          filename="package://rover_description/meshes/Arm_Stage_1.STL" />
-      </geometry>
-      <material
-        name="">
-        <color
-          rgba="0.752941176470588 0.752941176470588 0.752941176470588 1" />
-      </material>
-    </visual>
-    <collision>
-      <origin
-        xyz="0 0 0"
-        rpy="0 0 0" />
-      <geometry>
-        <mesh
-          filename="package://rover_description/meshes/Arm_Stage_1.STL" />
+          filename="package://rover_description/meshes/coarse/Arm_Stage_1.STL" />
+      </geometry>
+      <material
+        name="">
+        <color
+          rgba="0.752941176470588 0.752941176470588 0.752941176470588 1" />
+      </material>
+    </visual>
+    <collision>
+      <origin
+        xyz="0 0 0"
+        rpy="0 0 0" />
+      <geometry>
+        <mesh
+          filename="package://rover_description/meshes/coarse/Arm_Stage_1.STL" />
       </geometry>
     </collision>
@@ -377,19 +377,19 @@
       <geometry>
         <mesh
-          filename="package://rover_description/meshes/Arm_Stage_2.STL" />
-      </geometry>
-      <material
-        name="">
-        <color
-          rgba="0.752941176470588 0.752941176470588 0.752941176470588 1" />
-      </material>
-    </visual>
-    <collision>
-      <origin
-        xyz="0 0 0"
-        rpy="0 0 0" />
-      <geometry>
-        <mesh
-          filename="package://rover_description/meshes/Arm_Stage_2.STL" />
+          filename="package://rover_description/meshes/coarse/Arm_Stage_2.STL" />
+      </geometry>
+      <material
+        name="">
+        <color
+          rgba="0.752941176470588 0.752941176470588 0.752941176470588 1" />
+      </material>
+    </visual>
+    <collision>
+      <origin
+        xyz="0 0 0"
+        rpy="0 0 0" />
+      <geometry>
+        <mesh
+          filename="package://rover_description/meshes/coarse/Arm_Stage_2.STL" />
       </geometry>
     </collision>
@@ -428,19 +428,19 @@
       <geometry>
         <mesh
-          filename="package://rover_description/meshes/Arm_Stage_3.STL" />
-      </geometry>
-      <material
-        name="">
-        <color
-          rgba="0.752941176470588 0.752941176470588 0.752941176470588 1" />
-      </material>
-    </visual>
-    <collision>
-      <origin
-        xyz="0 0 0"
-        rpy="0 0 0" />
-      <geometry>
-        <mesh
-          filename="package://rover_description/meshes/Arm_Stage_3.STL" />
+          filename="package://rover_description/meshes/coarse/Arm_Stage_3.STL" />
+      </geometry>
+      <material
+        name="">
+        <color
+          rgba="0.752941176470588 0.752941176470588 0.752941176470588 1" />
+      </material>
+    </visual>
+    <collision>
+      <origin
+        xyz="0 0 0"
+        rpy="0 0 0" />
+      <geometry>
+        <mesh
+          filename="package://rover_description/meshes/coarse/Arm_Stage_3.STL" />
       </geometry>
     </collision>
@@ -479,19 +479,19 @@
       <geometry>
         <mesh
-          filename="package://rover_description/meshes/Arm_Stage_4.STL" />
-      </geometry>
-      <material
-        name="">
-        <color
-          rgba="0.752941176470588 0.752941176470588 0.752941176470588 1" />
-      </material>
-    </visual>
-    <collision>
-      <origin
-        xyz="0 0 0"
-        rpy="0 0 0" />
-      <geometry>
-        <mesh
-          filename="package://rover_description/meshes/Arm_Stage_4.STL" />
+          filename="package://rover_description/meshes/coarse/Arm_Stage_4.STL" />
+      </geometry>
+      <material
+        name="">
+        <color
+          rgba="0.752941176470588 0.752941176470588 0.752941176470588 1" />
+      </material>
+    </visual>
+    <collision>
+      <origin
+        xyz="0 0 0"
+        rpy="0 0 0" />
+      <geometry>
+        <mesh
+          filename="package://rover_description/meshes/coarse/Arm_Stage_4.STL" />
       </geometry>
     </collision>
@@ -530,19 +530,19 @@
       <geometry>
         <mesh
-          filename="package://rover_description/meshes/Arm_Gripper.STL" />
-      </geometry>
-      <material
-        name="">
-        <color
-          rgba="0.752941176470588 0.752941176470588 0.752941176470588 1" />
-      </material>
-    </visual>
-    <collision>
-      <origin
-        xyz="0 0 0"
-        rpy="0 0 0" />
-      <geometry>
-        <mesh
-          filename="package://rover_description/meshes/Arm_Gripper.STL" />
+          filename="package://rover_description/meshes/coarse/Arm_Gripper.STL" />
+      </geometry>
+      <material
+        name="">
+        <color
+          rgba="0.752941176470588 0.752941176470588 0.752941176470588 1" />
+      </material>
+    </visual>
+    <collision>
+      <origin
+        xyz="0 0 0"
+        rpy="0 0 0" />
+      <geometry>
+        <mesh
+          filename="package://rover_description/meshes/coarse/Arm_Gripper.STL" />
       </geometry>
     </collision>

Commit message: Update URDF and moveit joint positions and limits

File: rover_description/urdf/rover.control.xacro (robot description, xacro)
@@ -109,5 +109,5 @@
         <!-- <command_interface name="velocity"/> -->
         <param name="topic_name">base_rotate</param>
-        <param name="tick_resolution">-160000.0</param>
+        <param name="tick_resolution">-80000.0</param>
       </joint>
     </ros2_control>

File: rover_description/urdf/rover.urdf.xacro (robot description, xacro)
@@ -304,4 +304,9 @@
     <axis
       xyz="0 1 0" />
+    <limit
+      lower="-2.3562"
+      upper="2.3562"
+      velocity="0.25"
+      />
   </joint>
   <link name="Arm_Stage_1">
@@ -348,5 +353,5 @@
     <origin
       xyz="0 -0.010001 0"
-      rpy="0.7854 0 0" />
+      rpy="0 0 0" />
     <parent
       link="Arm_Base" />
@@ -355,4 +360,9 @@
     <axis
       xyz="1 0 0" />
+    <limit
+      lower="-1.5708"
+      upper="1.0472"
+      velocity="0.25"
+      />
   </joint>
   <link name="Arm_Stage_2">
@@ -399,5 +409,5 @@
     <origin
       xyz="0 0.52949 0"
-      rpy="-1.5708 0 -3.1416" />
+      rpy="0 3.1416 0" />
     <parent
       link="Arm_Stage_1" />
@@ -406,4 +416,9 @@
     <axis
       xyz="1 0 0" />
+    <limit
+      lower="-2.3562"
+      upper="2.3562"
+      velocity="0.5"
+      /> <!-- really vel should be 1.2 -->
   </joint>
   <link name="Arm_Stage_3">
@@ -457,4 +472,9 @@
     <axis
       xyz="0 1 0" />
+    <limit
+      lower="-3.1416"
+      upper="3.1416"
+      velocity="0.5"
+      /> <!-- really vel should be 1.2 -->
   </joint>
   <link name="Arm_Stage_4">
@@ -501,5 +521,5 @@
     <origin
       xyz="0 0.12103 0"
-      rpy="-0.7854 0 0" />
+      rpy="0 0 0" />
     <parent
       link="Arm_Stage_3" />
@@ -508,4 +528,9 @@
     <axis
       xyz="1 0 0" />
+    <limit
+      lower="-1.5708"
+      upper="1.5708"
+      velocity="0.5"
+      /> <!-- really vel should be 1.2 -->
   </joint>
   <link name="Arm_Gripper">
@@ -559,4 +584,9 @@
     <axis
       xyz="0 1 0" />
+    <limit
+      lower="-3.1416"
+      upper="3.1416"
+      velocity="0.5"
+      /> <!-- really vel should be 1.2 -->
   </joint>
   <xacro:rover_ros2_control use_gazebo="$(arg use_gazebo)"/>
